File: Buck_Practice/BuckPractice1.kicad_pcb (KiCad board)
At the start: 2 copper layers, 53 x 59 mm, 16 parts, among them J1 Screw_Terminal_01x02, J3 Screw_Terminal_01x02, Q1 FDMT80060DC, U2 LM25085MM

Commit message: hello 2
Parts:
- moved TP1 1.00 mm to (74.5, 108.5)
Routing:
- net Net-(U2-RT): track 33.2 -> 32.2 mm
Changed lines of the file:
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@@
 	(footprint "TestPoint:TestPoint_Pad_D1.0mm"
 		(layer "F.Cu")
-		(at 74.5 107.5)
+		(at 74.5 108.5)
 		(descr "SMD pad as test Point, diameter 1.0mm")
 		(tags "test point SMD pad")
@@
 	)
 	(via
-		(at 74.5 107.5)
+		(at 74.5 108.511166)
 		(size 0.6)
 		(drill 0.3)
@@
 	)
 	(segment
-		(start 75.488834 109.5)
-		(end 91 109.5)
+		(start 74.5 108.511166)
+		(end 75.488834 109.5)
 		(width 0.2)
 		(layer "B.Cu")
@@
 	)
 	(segment
-		(start 91 109.5)
-		(end 94.0875 106.4125)
+		(start 75.488834 109.5)
+		(end 91 109.5)
 		(width 0.2)
 		(layer "B.Cu")
@@
 	)
 	(segment
-		(start 74.5 108.511166)
-		(end 75.488834 109.5)
-		(width 0.2)
-		(layer "B.Cu")
-		(net 8)
-	)
-	(segment
-		(start 74.5 107.5)
-		(end 74.5 108.511166)
+		(start 91 109.5)
+		(end 94.0875 106.4125)
 		(width 0.2)
 		(layer "B.Cu")
