File: Boost_Practice/Maria/BoostPractice1.kicad_pcb (KiCad board)
At the start: 2 copper layers, 25 parts, among them J1 Screw_Terminal_2x5.08, J2 Screw_Terminal_2x5.08, Q1 IPB180N10S4-02, U1 LM3478MA

Commit message: Boost PCB Board
Parts:
- removed C2: C, rsx_capacitors:C_0805_2012Metric
- removed C3: C, Capacitor_SMD:C_Elec_10x10.2
- removed H1, H2, H3, H4: M4 PLATED, rsx_misc:MountingHole_4.5mm_Pad_Via
- removed R3: R, rsx_resistors:R_0805_2012Metric
- removed TP1, TP2, TP3, TP4: TestPoint_Small, TestPoint:TestPoint_Pad_D1.0mm
- added 4.7k101: R, rsx_resistors:R_0805_2012Metric, F.Cu at (136.8, 120.2)
- added C101: 100u, rsx_capacitors:C_0805_2012Metric, F.Cu at (107.5, 128.9)
- added D102: LED, LED_SMD:LED_0201_0603Metric_Pad0.64x0.40mm_HandSolder, F.Cu at (114.6, 122.3)
- added R101: 60k, rsx_resistors:R_0805_2012Metric, B.Cu at (133.0, 124.3)
- added SW101: SW_Nidec_CAS-120A1, Button_Switch_SMD:Nidec_Copal_CAS-120A, F.Cu at (119.5, 123.3)
- C1: value C -> 0.01u; footprint Capacitor_SMD:C_Elec_10x10.2 -> rsx_capacitors:C_0805_2012Metric
- C4: value C -> 100u
- C5: value C -> 22n
- L1: value L -> 10u
- R1: value R -> 0.025
- R2: value R -> 40k
- R4: value R -> 20k; moved to B.Cu
- U1: moved to B.Cu
- moved J2 88.3 mm to (141.6, 135.5)
- moved C1 82.2 mm to (132.9, 116.2)
- moved J1 75.7 mm to (104.8, 135.6)
- moved R4 72.8 mm to (131.8, 127.7), turned to -90 degrees
- moved F1 68.7 mm to (147.2, 120.8), turned to -90 degrees
- moved R2 68.6 mm to (115.0, 127.3), turned to -90 degrees
- moved R1 67.2 mm to (133.1, 112.0)
- moved C5 66.6 mm to (132.7, 121.2)
- moved C4 65.5 mm to (141.0, 109.2), turned to -90 degrees
- moved U1 60.5 mm to (126.4, 122.7), turned to 180 degrees
- moved Q1 53.4 mm to (121.6, 107.2), turned to 90 degrees
- moved D1 49.3 mm to (134.2, 102.6), turned to 180 degrees
- moved L1 41.2 mm to (108.5, 101.5), turned to 180 degrees
- moved F2 29.0 mm to (105.3, 118.6), turned to 90 degrees
Connections:
- C1 pad 1: unconnected-(C1-Pad1) -> /Isen
- C1 pad 2: unconnected-(C1-Pad2) -> GND
- C4 pad 1: unconnected-(C4-Pad1) -> /Vout_before_fuse
- C4 pad 2: unconnected-(C4-Pad2) -> GND
- C5 pad 1: unconnected-(C5-Pad1) -> /COMP
- C5 pad 2: unconnected-(C5-Pad2) -> Net-(4.7k101-Pad1)
- D1 pad 1: unconnected-(D1-K-Pad1) -> /Vout_before_fuse
- D1 pad 2: unconnected-(D1-A-Pad2) -> /V_ind
- F1 pad 1: unconnected-(F1-Pad1) -> /Vout_before_fuse
- F1 pad 2: unconnected-(F1-Pad2) -> /Vout
- F2 pad 1: unconnected-(F2-Pad1) -> /Vin
- F2 pad 2: unconnected-(F2-Pad2) -> /Vin_after_fuse
- J1 pad 1: unconnected-(J1-Pin_1-Pad1) -> /Vin
- J1 pad 2: unconnected-(J1-Pin_2-Pad2) -> GND
- J2 pad 1: unconnected-(J2-Pin_1-Pad1) -> GND
- J2 pad 2: unconnected-(J2-Pin_2-Pad2) -> /Vout
- L1 pad 1: unconnected-(L1-Pad1) -> /V_ind
- L1 pad 2: unconnected-(L1-Pad2) -> /Vin_after_fuse
- Q1 pad 1: unconnected-(Q1-G-Pad1) -> /DR
- Q1 pad 2: Net-(Q1-S-Pad2) -> /Isen
- Q1 pad 3: Net-(Q1-S-Pad2) -> /Isen
- Q1 pad 4: unconnected-(Q1-D-Pad4) -> /V_ind
- Q1 pad 5: Net-(Q1-S-Pad2) -> /Isen
- Q1 pad 6: Net-(Q1-S-Pad2) -> /Isen
- Q1 pad 7: Net-(Q1-S-Pad2) -> /Isen
- R1 pad 1: unconnected-(R1-Pad1) -> /Isen
- R1 pad 2: unconnected-(R1-Pad2) -> GND
- R2 pad 1: unconnected-(R2-Pad1) -> /V_boost_mode
- R2 pad 2: unconnected-(R2-Pad2) -> GND
- R4 pad 1: unconnected-(R4-Pad1) -> /V_FB
- R4 pad 2: unconnected-(R4-Pad2) -> GND
- U1 pad 1: unconnected-(U1-I_{SEN}-Pad1) -> /Isen
- U1 pad 2: unconnected-(U1-COMP-Pad2) -> /COMP
- U1 pad 3: unconnected-(U1-FB-Pad3) -> /V_FB
- U1 pad 4: unconnected-(U1-AGND-Pad4) -> GND
- U1 pad 5: unconnected-(U1-PGND-Pad5) -> GND
- U1 pad 6: unconnected-(U1-DR-Pad6) -> /DR
- U1 pad 7: unconnected-(U1-FA/SD-Pad7) -> /V_FA/SD
- U1 pad 8: unconnected-(U1-V_{IN}-Pad8) -> /Vin_after_fuse
Routing:
- net /Vout_before_fuse: vias 0 -> 1
- net /Vin_after_fuse: vias 0 -> 1
- added copper zone on F.Cu, net (none)
- added copper zone on F.Cu, net /Isen
- added copper zone on F.Cu, net /V_ind
- added copper zone on F.Cu, net /Vin_after_fuse
- added copper zone on F.Cu, net /Vout
- added copper zone on F.Cu, net /Vout_before_fuse
- added copper zone on B.Cu, net GND
- added copper zone on F.Cu, net GND
Other:
- board outline added: 57.5 x 49.2 mm
