File: Boost_Practice/Maria/BoostPractice1.kicad_sch (KiCad schematic)
At the start: 23 parts, among them J1 Screw_Terminal_2x5.08, J2 Screw_Terminal_2x5.08, Q1 IPB180N10S4-02, SW101 SW_Nidec_CAS-120A1, U1 LM3478MA

Commit message: Boost PCB Board
Parts:
- removed D101: LED, symbol Device:LED
- added D102: LED, LED_SMD:LED_0201_0603Metric_Pad0.64x0.40mm_HandSolder, symbol Device:LED
- renumbered 4.7k to 4.7k101
Connections:
- net V_LED_ON: now also D102.1 (K)
- net Vin_after_fuse: now also D102.2 (A)
Changed lines of the file:
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@@
 	(wire
 		(pts
-			(xy 41.91 82.55) (xy 85.09 82.55)
+			(xy 40.64 82.55) (xy 85.09 82.55)
 		)
 		(stroke
@@
 	(wire
 		(pts
-			(xy 41.91 82.55) (xy 41.91 100.33)
+			(xy 40.64 82.55) (xy 40.64 100.33)
 		)
 		(stroke
@@
 	(wire
 		(pts
-			(xy 49.53 100.33) (xy 64.77 100.33)
+			(xy 48.26 100.33) (xy 64.77 100.33)
 		)
 		(stroke
@@
 	)
 	(symbol
+		(lib_id "Device:LED")
+		(at 44.45 100.33 180)
+		(unit 1)
+		(exclude_from_sim no)
+		(in_bom yes)
+		(on_board yes)
+		(dnp no)
+		(fields_autoplaced yes)
+		(property "Reference" "D102"
+			(at 46.0375 92.71 0)
+			(effects
+				(font
+					(size 1.27 1.27)
+				)
+			)
+		)
+		(property "Value" "LED"
+			(at 46.0375 95.25 0)
+			(effects
+				(font
+					(size 1.27 1.27)
+				)
+			)
+		)
+		(property "Footprint" "LED_SMD:LED_0201_0603Metric_Pad0.64x0.40mm_HandSolder"
+			(at 44.45 100.33 0)
+			(effects
+				(font
+					(size 1.27 1.27)
+				)
+				(hide yes)
+			)
+		)
+		(property "Datasheet" "~"
+			(at 44.45 100.33 0)
+			(effects
+				(font
+					(size 1.27 1.27)
+				)
+				(hide yes)
+			)
+		)
+		(property "Description" "Light emitting diode"
+			(at 44.45 100.33 0)
+			(effects
+				(font
+					(size 1.27 1.27)
+				)
+				(hide yes)
+			)
+		)
+		(property "Sim.Pins" "1=K 2=A"
+			(at 44.45 100.33 0)
+			(effects
+				(font
+					(size 1.27 1.27)
+				)
+				(hide yes)
+			)
+		)
+		(pin "2"
+		)
+		(pin "1"
+		)
+		(instances
+			(project ""
+				(path "/bdacd1db-f779-4626-91d7-f5d5789723b2"
+					(reference "D102")
+					(unit 1)
+				)
+			)
+		)
+	)
+	(symbol
 		(lib_id "power:GND")
 		(at 118.11 83.82 0)
@@
 	)
 	(symbol
-		(lib_id "Device:LED")
-		(at 45.72 100.33 180)
-		(unit 1)
-		(exclude_from_sim no)
-		(in_bom yes)
-		(on_board yes)
-		(dnp no)
-		(fields_autoplaced yes)
-		(property "Reference" "D101"
-			(at 47.3075 92.71 0)
-			(effects
-				(font
-					(size 1.27 1.27)
-				)
-			)
-		)
-		(property "Value" "LED"
-			(at 47.3075 95.25 0)
-			(effects
-				(font
-					(size 1.27 1.27)
-				)
-			)
-		)
-		(property "Footprint" ""
-			(at 45.72 100.33 0)
-			(effects
-				(font
-					(size 1.27 1.27)
-				)
-				(hide yes)
-			)
-		)
-		(property "Datasheet" "~"
-			(at 45.72 100.33 0)
-			(effects
-				(font
-					(size 1.27 1.27)
-				)
-				(hide yes)
-			)
-		)
-		(property "Description" "Light emitting diode"
-			(at 45.72 100.33 0)
-			(effects
-				(font
-					(size 1.27 1.27)
-				)
-				(hide yes)
-			)
-		)
-		(pin "2"
-		)
-		(pin "1"
-		)
-		(instances
-			(project ""
-				(path "/bdacd1db-f779-4626-91d7-f5d5789723b2"
-					(reference "D101")
-					(unit 1)
-				)
-			)
-		)
-	)
-	(symbol
 		(lib_id "Device:L")
 		(at 130.81 82.55 180)
@@
 		(dnp no)
 		(fields_autoplaced yes)
-		(property "Reference" "4.7k"
+		(property "Reference" "4.7k101"
 			(at 87.63 126.9999 0)
 			(effects
@@
 			(project "BoostPractice1"
 				(path "/bdacd1db-f779-4626-91d7-f5d5789723b2"
-					(reference "4.7k")
+					(reference "4.7k101")
 					(unit 1)
 				)

Commit message: testing 123
Parts:
- removed H1, H2: M4 PLATED, rsx_misc:MountingHole_4.5mm_Pad_Via, symbol rsx_misc:M4 PLATED
Changed lines of the file:
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@@
-	)
-	(symbol
-		(lib_id "rsx_misc:M4 PLATED")
-		(at 227.33 100.33 0)
-		(unit 1)
-		(exclude_from_sim no)
-		(in_bom no)
-		(on_board yes)
-		(dnp no)
-		(fields_autoplaced yes)
-		(property "Reference" "H1"
-			(at 229.87 97.7899 0)
-			(effects
-				(font
-					(size 1.27 1.27)
-				)
-				(justify left)
-			)
-		)
-		(property "Value" "M4 PLATED"
-			(at 229.87 100.3299 0)
-			(effects
-				(font
-					(size 1.27 1.27)
-				)
-				(justify left)
-			)
-		)
-		(property "Footprint" "rsx_misc:MountingHole_4.5mm_Pad_Via"
-			(at 227.33 100.33 0)
-			(effects
-				(font
-					(size 1.27 1.27)
-				)
-				(hide yes)
-			)
-		)
-		(property "Datasheet" "~"
-			(at 227.33 100.33 0)
-			(effects
-				(font
-					(size 1.27 1.27)
-				)
-				(hide yes)
-			)
-		)
-		(property "Description" "Mounting Hole with connection M4"
-			(at 227.33 100.33 0)
-			(effects
-				(font
-					(size 1.27 1.27)
-				)
-				(hide yes)
-			)
-		)
-		(pin "1"
-		)
-		(instances
-			(project "BoostPractice1"
-				(path "/bdacd1db-f779-4626-91d7-f5d5789723b2"
-					(reference "H1")
-					(unit 1)
-				)
-			)
-		)
 	)
 	(symbol
@@
 					(unit 1)
 				)
-			)
-		)
-	)
-	(symbol
-		(lib_id "rsx_misc:M4 PLATED")
-		(at 227.33 115.57 0)
-		(unit 1)
-		(exclude_from_sim no)
-		(in_bom no)
-		(on_board yes)
-		(dnp no)
-		(fields_autoplaced yes)
-		(property "Reference" "H2"
-			(at 229.87 113.0299 0)
-			(effects
-				(font
-					(size 1.27 1.27)
-				)
-				(justify left)
-			)
-		)
-		(property "Value" "M4 PLATED"
-			(at 229.87 115.5699 0)
-			(effects
-				(font
-					(size 1.27 1.27)
-				)
-				(justify left)
-			)
-		)
-		(property "Footprint" "rsx_misc:MountingHole_4.5mm_Pad_Via"
-			(at 227.33 115.57 0)
-			(effects
-				(font
-					(size 1.27 1.27)
-				)
-				(hide yes)
-			)
-		)
-		(property "Datasheet" "~"
-			(at 227.33 115.57 0)
-			(effects
-				(font
-					(size 1.27 1.27)
-				)
-				(hide yes)
-			)
-		)
-		(property "Description" "Mounting Hole with connection M4"
-			(at 227.33 115.57 0)
-			(effects
-				(font
-					(size 1.27 1.27)
-				)
-				(hide yes)
-			)
-		)
-		(pin "1"
-		)
-		(instances
-			(project "BoostPractice1"
-				(path "/bdacd1db-f779-4626-91d7-f5d5789723b2"
-					(reference "H2")
-					(unit 1)
-				)
