File: Buck_Practice/Rivera/BuckPractice.kicad_sch (KiCad schematic)
At the start: 32 parts, among them J1 Screw_Terminal_2x5.08, J2 Screw_Terminal_2x5.08, Q102 QM6015D, SW101 SW_SPST, SW102 SW_SPST, U101 LM25085MM

Commit message: update1
Parts:
- R4: value R -> 3.4k
Changed lines of the file:
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@@
 			)
 		)
-		(property "Value" "R"
+		(property "Value" "3.4k"
 			(at 194.31 123.1899 0)
 			(effects

Commit message: update
Parts:
- removed C7: C, rsx_capacitors:C_0805_2012Metric, symbol rsx_Capacitors:1u
- removed F2: Fuse_Holder_Auto, rsx_fuses:FUSE_3568-10, symbol rsx_fuses:Fuse_Holder_Auto
- removed SW101: SW_SPST, symbol Switch:SW_SPST
- removed TP1, TP2, TP3, TP4: TestPoint_Small, TestPoint:TestPoint_Pad_D1.0mm, symbol rsx_misc:TestPoint_Small
- R6: renamed from R4; value 3.4k -> R
- renumbered C6 to C1, C5 to C2, C2 to C3, C1 to C4, C3 to C5, C101 to C6, C4 to C7, D2 to D1, Q102 to Q1, R101 to R3, R102 to R4, R3 to R5, SW102 to SW1, U101 to U1
Connections:
- net Vin: now also F1.1; no longer C1.1, C2.1, C3.1, C4.1, R1.2, R2.1, R3.2, U1.8 (VIN)
- net at F1.2: now also C1.1, C2.1, C3.1, C4.1, R1.2, R2.1, R3.2, U1.8 (VIN)
Other:
- note removed: "Electrolytic Capacitors"
- note removed: "Passive Capacitors"
- note removed: "Passive Resistors"
- note removed: "Power Diode"
- note removed: "Terminal Input/Output + Fuses"
- note removed: "Test Points"
- moved on the sheet: F1

Commit message: final for now
Parts:
- R6: value R -> 3.4k
Changed lines of the file:
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@@
 			)
 		)
-		(property "Value" "R"
+		(property "Value" "3.4k"
 			(at 194.31 123.1899 0)
 			(effects
