File: Buck_Practice/Rivera/BuckPractice.kicad_pcb (KiCad board)
At the start: 2 copper layers, 24 parts, among them J1 Screw_Terminal_2x5.08, J2 Screw_Terminal_2x5.08, Q102 QM6015D, U101 LM25085MM

Commit message: final update
Parts:
- added SW1: SW_SPST, Connector_PinHeader_2.54mm:PinHeader_1x02_P2.54mm_Vertical, F.Cu at (147.0, 123.0)
- R6: renamed from R4; value R -> 3.4k
- moved H1 61.5 mm to (175.2, 122.5)
- moved J1 59.5 mm to (122.2, 123.2)
- moved R1 49.6 mm to (145.2, 116.5), turned to 180 degrees
- moved R2 44.2 mm to (144.5, 112.8), turned to -90 degrees
- moved R5 43.7 mm to (152.5, 119.2), turned to 180 degrees
- moved R6 43.5 mm to (152.5, 122.0)
- moved H2 41.3 mm to (175.0, 95.0)
- moved C4 37.1 mm to (141.8, 112.8), turned to -90 degrees
- moved C2 36.2 mm to (142.0, 117.5), turned to -90 degrees
- moved C7 35.6 mm to (164.2, 120.2), turned to -90 degrees
- moved H3 32.1 mm to (114.3, 122.6)
- moved J2 31.7 mm to (174.5, 111.8), turned to 90 degrees
- moved C5 31.1 mm to (150.5, 116.5), turned to 180 degrees
- moved R3 30.2 mm to (151.2, 109.2), turned to -90 degrees
- moved R4 29.9 mm to (153.0, 113.0), turned to 180 degrees
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- renumbered C6 to C1, C5 to C2, C2 to C3, C1 to C4, C3 to C5, C101 to C6, C4 to C7, D2 to D1, Q102 to Q1, R101 to R3, R102 to R4, R3 to R5, U101 to U1
Connections:
- J1 pad 1: /Vin -> GND
- J1 pad 2: GND -> /Vin
Routing:
- net Net-(U1-FB): track 0.00 -> 9.99 mm
- net Net-(SW1-B): track 0.00 -> 8.11 mm
- net Net-(C5-Pad1): track 0.00 -> 6.36 mm
- net Net-(Q1-S): track 0.00 -> 5.66 mm
- net Net-(Q1-G): track 0.00 -> 3.20 mm
- net GND: track 0.00 -> 1.24 mm, vias 0 -> 15
- added copper zone on F.Cu, net /Vin
- added copper zone on F.Cu, net /Vout
- added copper zone on B.Cu, net GND
- added copper zone on F.Cu, net GND
- added copper zone on F.Cu, net Net-(D1-K)
- added copper zone on F.Cu, net Net-(U1-ADJ)
- added copper zone on F.Cu, net Net-(U1-VCC)
- added copper zone on F.Cu, net Net-(U1-VIN)
Other:
- board outline added: 76 x 44 mm
