File: 4_switch_Buck_Boost/Buck_Boost_main.kicad_sch (KiCad schematic)
At the start: 71 parts, among them J1 Screw_Terminal_2x5.08, J2 Screw_Terminal_2x5.08, J3 Screw_Terminal_2x2.54, Q1 CSD18532Q5B, Q101 2N7002K, Q103 BSS83P, Q2 CSD18532Q5B, Q3 CSD18532Q5B, Q4 CSD18532Q5B, U1 LT8390EUFD_PBF

Commit message: final schem
Parts:
- removed C125: C, rsx_capacitors:C_0603_1608Metric, symbol Device:C
- removed C126: C, rsx_capacitors:C_0805_2012Metric, symbol Device:C
- removed C127: C, rsx_capacitors:C_2220_5750Metric_Pad1.97x5.40mm_HandSolder, symbol Device:C
- removed C128: C_Polarized, Capacitor_SMD:CP_Elec_8x10.5, symbol Device:C_Polarized
- removed R119: R_Shunt, Resistor_SMD:R_Shunt_Vishay_WSK2512_6332Metric_T1.19mm, symbol Device:R_Shunt
- removed R120: R, rsx_resistors:R_0603_1608Metric, symbol Device:R
- removed R121: R, rsx_resistors:R_1206_3216Metric, symbol Device:R
- C104, C105: value 2.5u -> 0.47u
- C5: footprint (none) -> rsx_capacitors:C_0603_1608Metric
- R101: value 5.5m -> 6m; footprint Resistor_SMD:R_Shunt_Vishay_WSK2512_6332Metric_T1.19mm -> Resistor_SMD:R_Shunt_Vishay_WSR2_WSR3
- R102: value 10m -> 15m; footprint Resistor_SMD:R_Shunt_Vishay_WSK2512_6332Metric_T1.19mm -> Resistor_SMD:R_Shunt_Vishay_WSR2_WSR3
Connections:
- net EN/UVLO: no longer U1.8 (LOADEN)
- net GND: now also C5.2, R104.2
- net at C103.2, U1.10 (CTRL), U1.9 (VREF): now also U1.8 (LOADEN)
Other:
- note removed: "selection of diff res, with diff footprints"
- note removed: "shunt 603 1206 603 805 2220 polar"
- moved on the sheet: C104, C105, C5, F1

Commit message: Updated Schematic with cool stuff trust
Parts:
- removed C104, C105: 0.47u, rsx_capacitors:C_0603_1608Metric, symbol Device:C
- removed C122: 4.7u, rsx_capacitors:C_0805_2012Metric, symbol Device:C
- removed C130: 22n, rsx_capacitors:C_0603_1608Metric, symbol Device:C
- removed D101: LED_G, rsx_leds:LED_0805_2012Metric, symbol rsx_LEDs:LED_G
- removed HW1: Board_Mount_Heat_Sink_Screw_2.5C/W, rsx_misc:ATS-1139-C1-R0, symbol rsx_misc:Board_Mount_Heat_Sink_Screw_2.5C/W
- removed J1: Screw_Terminal_2x5.08, rsx_headers_screw:Molex_0398800302, symbol rsx_header_screw:Screw_Terminal_2x5.08
- removed R101: 6m, Resistor_SMD:R_Shunt_Vishay_WSR2_WSR3, symbol Device:R_Shunt
- removed R102: 15m, Resistor_SMD:R_Shunt_Vishay_WSR2_WSR3, symbol Device:R_Shunt
- removed R108: 4.7k, rsx_resistors:R_0603_1608Metric, symbol Device:R
- added C1: 4.7u, rsx_capacitors:C_0805_2012Metric, symbol Device:C
- added C4: 22n, rsx_capacitors:C_0603_1608Metric, symbol Device:C
- added C6, C7: 1.0u, rsx_capacitors:C_0805_2012Metric, symbol Device:C
- added C8, C9: 0.47u, rsx_capacitors:C_0603_1608Metric, symbol Device:C
- added D1, D2, D3: LED_G, rsx_leds:LED_0805_2012Metric, symbol rsx_LEDs:LED_G
- added F3: 40mm_by_20mm_Fan_Vertical, rsx_misc:40mmFan, symbol rsx_misc:40mm_by_40mm_Fan_Mount_Vertical
- added H1, H2, H3, H4: M4 PLATED, MountingHole:MountingHole_3.2mm_M3_Pad_Via, symbol rsx_misc:M4 PLATED
- added HW2: Board_Mount_Heat_Sink_Adhesive, rsx_misc:BDN10-3CB_A01, symbol rsx_misc:Board_Mount_Heat_Sink_Adhesive
- added J1: Conn_02x02_Counter_Clockwise, Connector_PinHeader_1.00mm:PinHeader_2x02_P1.00mm_Vertical, symbol Connector_Generic:Conn_02x02_Counter_Clockwise
- added J4: Screw_Terminal_2x5.08, rsx_headers_screw:Molex_0398800302, symbol rsx_header_screw:Screw_Terminal_2x5.08
- added M1: Fan, Connector_Molex:Molex_KK-396_5273-02A_1x02_P3.96mm_Vertical, symbol Motor:Fan
- added NT1: NetTie_2, rsx_misc:NetTie-2_SMD_Pad0.5mm, symbol rsx_misc:NetTie_2
- added Q6: AO3400A, Package_TO_SOT_SMD:SOT-23, symbol Transistor_FET:AO3400A
- added R1, R2, R3: 4.7k, rsx_resistors:R_0603_1608Metric, symbol Device:R
- added R10: 50k, rsx_resistors:R_0603_1608Metric, symbol Device:R
- added R4: 100K, rsx_resistors:R_0603_1608Metric, symbol Device:R
- added R5: 10k, rsx_resistors:R_0603_1608Metric, symbol Device:R
- added R6: 100, rsx_resistors:R_0603_1608Metric, symbol Device:R
- added R7: 6m, shunt:RES_KRL3216T4-M-R003-F-T1, symbol shunts:KRL3216T4-M-R003-F-T1
- added R8: 15m, shunt:RES_KRL3216T4-M-R003-F-T1, symbol shunts:KRL3216T4-M-R003-F-T1
- added R9: 300k, rsx_resistors:R_0603_1608Metric, symbol Device:R
- added TH1: 10k, Connector_Molex:Molex_KK-396_5273-02A_1x02_P3.96mm_Vertical, symbol rsx_sensors:NTCALUG54A103G351A
- added TP1: BAT, TestPoint:TestPoint_2Pads_Pitch2.54mm_Drill0.8mm, symbol Connector:TestPoint_2Pole
- added TP10: EN, TestPoint:TestPoint_Pad_D1.0mm, symbol Connector:TestPoint
- added TP11: Output, TestPoint:TestPoint_2Pads_Pitch2.54mm_Drill0.8mm, symbol Connector:TestPoint_2Pole
- added TP12, TP2, TP9: GND, TestPoint:TestPoint_Pad_D1.0mm, symbol Connector:TestPoint
- added TP13: GNDA, TestPoint:TestPoint_Pad_D1.0mm, symbol Connector:TestPoint
- added TP3: SW1, TestPoint:TestPoint_Loop_D1.80mm_Drill1.0mm_Beaded, symbol Connector:TestPoint
- added TP4: SW2, TestPoint:TestPoint_Loop_D1.80mm_Drill1.0mm_Beaded, symbol Connector:TestPoint
- added TP5: RT, TestPoint:TestPoint_Pad_D1.0mm, symbol Connector:TestPoint
- added TP6: FB, TestPoint:TestPoint_Pad_D1.0mm, symbol Connector:TestPoint
- added TP7: Vout, TestPoint:TestPoint_Pad_D1.0mm, symbol Connector:TestPoint
- added TP8: Vin, TestPoint:TestPoint_Pad_D1.0mm, symbol Connector:TestPoint
- C101, C106: value 0.1u -> 4.7u; footprint rsx_capacitors:C_0603_1608Metric -> rsx_capacitors:C_0805_2012Metric
- C102: value 1u -> 0.1u
- C107, C108, C117: value 33u -> 47u
- C109, C110, C111: value 22u -> 33u
- C114, C115, C116: footprint rsx_capacitors:C_0805_2012Metric -> rsx_capacitors:C_0603_1608Metric
- C123, C124: footprint rsx_capacitors:C_0603_1608Metric -> Capacitor_SMD:C_0805_2012Metric
- C129: value 4.7n -> 0.1u
- C131: value 4.7n -> 22n
- F1, F2: footprint rsx_fuses:FUSE_3568-10 -> Fuse:Fuseholder_Blade_Mini_Keystone_3568
- L1: footprint rsx_inductors:PQ2617BHA-XXXK -> Inductor_SMD:L_Wuerth_WE-XHMI-8080
- R104: value 5k -> 10k
- R107, R109: value 10K -> 100K
- R113, R114: footprint rsx_resistors:R_0603_1608Metric -> Capacitor_SMD:C_0805_2012Metric
- RV101, RV102: footprint rsx_resistors:Potentiometer_Bourns_3296W_Vertical_DL -> Potentiometer_SMD:Potentiometer_Bourns_3314G_Vertical
Connections:
- net BAT: now also J2.1 (Pin_1), TP1.2
- net ENABLE: now also TP10.1
- net EN/UVLO: now also R10.1, R3.1, R9.2; no longer C115.1, Q103.3 (D), R107.1
- net FB: now also TP6.1
- net GND: now also C4.2, C6.1, C7.1, D1.1 (K), D2.1 (K), D3.1 (K), F3.1, H1.1, H2.1, H3.1, H4.1, J4.2 (Pin_2), NT1.2, Q6.2 (S), R4.2, TH1.2, TP1.1, TP11.1, TP12.1, TP2.1, TP9.1; no longer C103.1, C119.2, C120.2, C121.2, C5.2, R104.2, RV101.2, RV101.3, U1.7 (TEST)
- net ISN: now also R8.1
- net ISP: now also R8.4
- net LSN: now also R7.4
- net LSP: now also R7.1
- net Vin: now also C4.1, C6.2, R1.1, TP8.1
- net Vout: now also C7.2, R8.3, TP7.1
- net Vref: now reaches C103.2, U1.10 (CTRL), U1.8 (LOADEN), U1.9 (VREF)
- net OUTPUT: now reaches F2.1
- net OUTPUT: now also J4.1 (Pin_1), M1.1 (+), R5.1, TP11.2; no longer J2.1 (Pin_1)
- net at U1.27 (BST1): now also C8.1
- net at L1.1: now also R7.3
- net at U1.24 (BST2): now also C9.1
- net at R111.2, U1.18 (RT): now also TP5.1
- net INTVCC: now reaches R112.2, U1.5 (INTVCC)
- net INTVCC: now also C1.2, J1.2 (Pin_2); no longer U1.19 (SYNC/SPRD)
- net BST1 renamed SW1
- net SW1: now also C8.2, R7.2, TP3.1
- net BST2 renamed SW2
- net SW2: now also C9.2, TP4.1
- net Vout_fb renamed Vout_FB
- net Vout_FB: now also R2.1, R8.2
- new net: Q6.1 (G), R4.1, R6.1
- new net: C115.1, Q103.3 (D), R107.1, R9.1
- new net: R5.2, R6.2, TH1.1
- new net: D3.2 (A), R3.2
- new net: D2.2 (A), R2.2
- new net: D1.2 (A), R1.2
- new net: M1.2 (-), Q6.3 (D)
- new net GNDA: C1.1, C103.1, C119.2, C120.2, C121.2, C5.2, J1.1 (Pin_1), NT1.1, R10.2, R104.2, RV101.2, RV101.3, TP13.1, U1.7 (TEST)
- new net SYNC/SPRD: J1.3 (Pin_3), J1.4 (Pin_4), U1.19 (SYNC/SPRD)
Other:
- note added: "18-25.6V"
- note added: "24V"
- note added: "5A"
- note added: "6.7A - 4.7A"
- note added: ">= 1W"
- note added: "AUXILLIARY CIRCUITS"
- note added: "Adjusted for En/UVLO ~ Cannot recieve 24V directly ~1.3V Now"
- note added: "BULK CAP"
- note added: "CONTROLLER"
- note added: "ENABLE LEVEL SHIFTER"
- note added: "FB: 24V : ((200k+30k)+10k)/10k"
- note added: "FEEDBACK LOOP"
- note added: "Fan Control Using Heat Probe"
- note added: "For easier ripple probing (groung spring)"
- note added: "INPUT FILTER"
- note added: "LEDS/TERMINALS"
- note added: "MOUNTING HOLES/HEATSINK/FAN MOUNT"
- note added: "NTC FAN PORT CONTROL"
- note added: "OUTPUT FILTER"
- note added: "POWER STAGE"
- note added: "RT: 100kOhm -- 400kHz 75kOhm -- 500kHz 59kOhm -- 600kHz"
- note added: "Use Jumper Cap to choose triangle spread or internal osc"
- note added: "will likely adjust bypass filters"
- company: (none) -> Robotics for Space Exploration
- title: (none) -> 4-Switch Buck-Boost Converter 120W
- moved on the sheet: C101, C102, C103, C106, C107, C108, C109, C110, C111, C112, C113, C114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
